Commit message: Paquete de programas que ejecutan y ayudan a visualizar la IK para el brazo de aura

File: IK/g1_dual_arm_copy.urdf (robot description, URDF)
Before this commit: robot g1_dual_arm, 18 links, 17 joints
Links:
- removed link right_elbow_link
- removed link right_rubber_hand
- removed link right_shoulder_pitch_link
- removed link right_shoulder_roll_link
- removed link right_shoulder_yaw_link
- removed link right_wrist_pitch_link
- removed link right_wrist_roll_link
- removed link right_wrist_yaw_link
- added link left_elbow_link, mass 0.6; collision mesh filename=meshes/left_elbow_link.STL; visual mesh filename=meshes/left_elbow_link.STL
- added link left_rubber_hand, mass 0.170; visual mesh filename=meshes/left_rubber_hand.STL
- added link left_shoulder_pitch_link, mass 0.718; collision cylinder length=0.05 radius=0.03; visual mesh filename=meshes/left_shoulder_pitch_link.STL
- added link left_shoulder_roll_link, mass 0.643; collision cylinder length=0.03 radius=0.03; visual mesh filename=meshes/left_shoulder_roll_link.STL
- added link left_shoulder_yaw_link, mass 0.734; collision mesh filename=meshes/left_shoulder_yaw_link.STL; visual mesh filename=meshes/left_shoulder_yaw_link.STL
- added link left_wrist_pitch_link, mass 0.48404956; collision mesh filename=meshes/left_wrist_pitch_link.STL; visual mesh filename=meshes/left_wrist_pitch_link.STL
- added link left_wrist_roll_link, mass 0.08544498; collision mesh filename=meshes/left_wrist_roll_link.STL; visual mesh filename=meshes/left_wrist_roll_link.STL
- added link left_wrist_yaw_link, mass 0.08457647; collision mesh filename=meshes/left_wrist_yaw_link.STL; visual mesh filename=meshes/left_wrist_yaw_link.STL
Joints:
- removed joint right_elbow_joint
- removed joint right_hand_palm_joint
- removed joint right_shoulder_pitch_joint
- removed joint right_shoulder_roll_joint
- removed joint right_shoulder_yaw_joint
- removed joint right_wrist_pitch_joint
- removed joint right_wrist_roll_joint
- removed joint right_wrist_yaw_joint
- added joint left_elbow_joint: type revolute, parent left_shoulder_yaw_link, child left_elbow_link, origin xyz=0.015783 0 -0.080518 rpy=0 0 0, axis 0 1 0, limit lower=-1.0472 upper=2.0944 effort=25 velocity=37
- added joint left_hand_palm_joint: type fixed, parent left_wrist_yaw_link, child left_rubber_hand, origin xyz=0.0415 0.003 0 rpy=0 0 0
- added joint left_shoulder_pitch_joint: type revolute, parent torso_link, child left_shoulder_pitch_link, origin xyz=0.0039563 0.10022 0.23778 rpy=0.27931 5.4949E-05 -0.00019159, axis 0 1 0, limit lower=-3.0892 upper=2.6704 effort=25 velocity=37
- added joint left_shoulder_roll_joint: type revolute, parent left_shoulder_pitch_link, child left_shoulder_roll_link, origin xyz=0 0.038 -0.013831 rpy=-0.27925 0 0, axis 1 0 0, limit lower=-1.5882 upper=2.2515 effort=25 velocity=37
- added joint left_shoulder_yaw_joint: type revolute, parent left_shoulder_roll_link, child left_shoulder_yaw_link, origin xyz=0 0.00624 -0.1032 rpy=0 0 0, axis 0 0 1, limit lower=-2.618 upper=2.618 effort=25 velocity=37
- added joint left_wrist_pitch_joint: type revolute, parent left_wrist_roll_link, child left_wrist_pitch_link, origin xyz=0.038 0 0 rpy=0 0 0, axis 0 1 0, limit lower=-1.614429558 upper=1.614429558 effort=5 velocity=22
- added joint left_wrist_roll_joint: type revolute, parent left_elbow_link, child left_wrist_roll_link, origin xyz=0.100 0.00188791 -0.010 rpy=0 0 0, axis 1 0 0, limit lower=-1.972222054 upper=1.972222054 effort=25 velocity=37
- added joint left_wrist_yaw_joint: type revolute, parent left_wrist_pitch_link, child left_wrist_yaw_link, origin xyz=0.046 0 0 rpy=0 0 0, axis 0 0 1, limit lower=-1.614429558 upper=1.614429558 effort=5 velocity=22

Commit message: IK con brazo izquierdo

File: IK/g1_dual_arm_copy.urdf (robot description, URDF)
Before this commit: robot g1_dual_arm, 18 links, 17 joints
Links:
- removed link left_elbow_link
- removed link left_rubber_hand
- removed link left_shoulder_pitch_link
- removed link left_shoulder_roll_link
- removed link left_shoulder_yaw_link
- removed link left_wrist_pitch_link
- removed link left_wrist_roll_link
- removed link left_wrist_yaw_link
- added link right_elbow_link, mass 0.6; collision mesh filename=meshes/right_elbow_link.STL; visual mesh filename=meshes/right_elbow_link.STL
- added link right_rubber_hand, mass 0.170; visual mesh filename=meshes/right_rubber_hand.STL
- added link right_shoulder_pitch_link, mass 0.718; collision cylinder length=0.05 radius=0.03; visual mesh filename=meshes/right_shoulder_pitch_link.STL
- added link right_shoulder_roll_link, mass 0.643; collision cylinder length=0.03 radius=0.03; visual mesh filename=meshes/right_shoulder_roll_link.STL
- added link right_shoulder_yaw_link, mass 0.734; collision mesh filename=meshes/right_shoulder_yaw_link.STL; visual mesh filename=meshes/right_shoulder_yaw_link.STL
- added link right_wrist_pitch_link, mass 0.48404956; collision mesh filename=meshes/right_wrist_pitch_link.STL; visual mesh filename=meshes/right_wrist_pitch_link.STL
- added link right_wrist_roll_link, mass 0.08544498; collision mesh filename=meshes/right_wrist_roll_link.STL; visual mesh filename=meshes/right_wrist_roll_link.STL
- added link right_wrist_yaw_link, mass 0.08457647; collision mesh filename=meshes/right_wrist_yaw_link.STL; visual mesh filename=meshes/right_wrist_yaw_link.STL
Joints:
- removed joint left_elbow_joint
- removed joint left_hand_palm_joint
- removed joint left_shoulder_pitch_joint
- removed joint left_shoulder_roll_joint
- removed joint left_shoulder_yaw_joint
- removed joint left_wrist_pitch_joint
- removed joint left_wrist_roll_joint
- removed joint left_wrist_yaw_joint
- added joint right_elbow_joint: type revolute, parent right_shoulder_yaw_link, child right_elbow_link, origin xyz=0.015783 0 -0.080518 rpy=0 0 0, axis 0 1 0, limit lower=-1.0472 upper=2.0944 effort=25 velocity=37
- added joint right_hand_palm_joint: type fixed, parent right_wrist_yaw_link, child right_rubber_hand, origin xyz=0.0415 -0.003 0 rpy=0 0 0
- added joint right_shoulder_pitch_joint: type revolute, parent torso_link, child right_shoulder_pitch_link, origin xyz=0.0039563 -0.10021 0.23778 rpy=-0.27931 5.4949E-05 0.00019159, axis 0 1 0, limit lower=-3.0892 upper=2.6704 effort=25 velocity=37
- added joint right_shoulder_roll_joint: type revolute, parent right_shoulder_pitch_link, child right_shoulder_roll_link, origin xyz=0 -0.038 -0.013831 rpy=0.27925 0 0, axis 1 0 0, limit lower=-2.2515 upper=1.5882 effort=25 velocity=37
- added joint right_shoulder_yaw_joint: type revolute, parent right_shoulder_roll_link, child right_shoulder_yaw_link, origin xyz=0 -0.00624 -0.1032 rpy=0 0 0, axis 0 0 1, limit lower=-2.618 upper=2.618 effort=25 velocity=37
- added joint right_wrist_pitch_joint: type revolute, parent right_wrist_roll_link, child right_wrist_pitch_link, origin xyz=0.038 0 0 rpy=0 0 0, axis 0 1 0, limit lower=-1.614429558 upper=1.614429558 effort=5 velocity=22
- added joint right_wrist_roll_joint: type revolute, parent right_elbow_link, child right_wrist_roll_link, origin xyz=0.100 -0.00188791 -0.010 rpy=0 0 0, axis 1 0 0, limit lower=-1.972222054 upper=1.972222054 effort=25 velocity=37
- added joint right_wrist_yaw_joint: type revolute, parent right_wrist_pitch_link, child right_wrist_yaw_link, origin xyz=0.046 0 0 rpy=0 0 0, axis 0 0 1, limit lower=-1.614429558 upper=1.614429558 effort=5 velocity=22
